File: PCB/AirU/AirU.kicad_pcb (KiCad board)
At the start: 2 copper layers, 167 x 87.9 mm, 31 parts, among them IC3 LD1086DT50TR, J1 53261-7008, J2 ZX62-B-5PA_33_, U1 ESP32-S3-WROOM-1, U2 CH340E, U3 LoRa_Breakout, U4 MICS6814, U5 HDC2010YPAR

Commit message: pcb layout complete
Parts:
- added J3: Conn_01x02_Male, Connector_PinHeader_2.54mm:PinHeader_1x02_P2.54mm_Vertical, F.Cu at (160.1, 41.7)
- added J4: Conn_01x02_Male, Connector_PinHeader_2.54mm:PinHeader_1x02_P2.54mm_Vertical, F.Cu at (183.0, 57.2)
- added J5: Conn_01x01_Male, Connector_PinHeader_2.54mm:PinHeader_1x01_P2.54mm_Vertical, F.Cu at (136.1, 27.2)
- added J6: Conn_01x02_Male, Connector_PinHeader_2.54mm:PinHeader_1x02_P2.54mm_Vertical, F.Cu at (171.0, 52.1)
- added REF**: MountingHole_2.7mm_M2.5_DIN965_Pad, MountingHole:MountingHole_2.7mm_M2.5_DIN965_Pad, F.Cu at (194.6, 57.1)
- moved R16 57.5 mm to (123.7, 45.3), turned to 0 degrees
- moved U5 54.4 mm to (132.7, 41.6)
- moved R15 54.2 mm to (132.9, 43.8), turned to 180 degrees
- moved IC3 52.3 mm to (126.5, 47.4)
- moved U4 37.4 mm to (138.8, 36.8)
- moved R12 36.9 mm to (140.2, 28.7), turned to 90 degrees
- moved C2 35.6 mm to (132.0, 54.9), turned to 90 degrees
- moved R13 23.0 mm to (132.3, 34.4), turned to -90 degrees
- moved U3 13.0 mm to (185.6, 31.8)
- moved R14 11.9 mm to (132.1, 51.6), turned to -90 degrees
- moved D1 7.84 mm to (123.0, 42.9), turned to 90 degrees
- moved J2 0.15 mm to (128.2, 25.3)
Connections:
- U4 pad 8: /GPIO18 -> /GPIO8
Routing:
- net GND: track 73.9 -> 211.6 mm, vias 0 -> 2
- net VDD: track 62.9 -> 158.8 mm, vias 0 -> 7
- net /GPIO18: track 0.00 -> 71.8 mm, vias 0 -> 4
- net /U0RXD: track 0.00 -> 64.4 mm, vias 0 -> 4
- net VCC: track 7.71 -> 72.1 mm, vias 0 -> 5
- net /U0TXD: track 3.60 -> 65.1 mm, vias 1 -> 4
- net /GPIO8: track 0.00 -> 46.4 mm, vias 0 -> 2
- net /GPIO16: track 0.00 -> 37.4 mm, vias 0 -> 2
- net /GPIO17: track 0.00 -> 34.2 mm, vias 0 -> 2
- net /GPIO5: track 0.00 -> 31.2 mm, vias 0 -> 2
- net /GPIO19: track 0.00 -> 29.4 mm, vias 0 -> 4
- net /GPIO45: track 6.29 -> 33.3 mm, vias 0 -> 2
- net /GPIO14: track 0.00 -> 26.5 mm
- net /GPIO13: track 0.00 -> 24.1 mm
- net /GPIO48: track 0.00 -> 22.1 mm, vias 0 -> 2
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- added copper zone on F.Cu, net GND
Other:
- board size 167 x 87.9 mm -> 77.7 x 40.3 mm
- board text added: "LoRaWAN AirU Demo Board v1 Michael Keyser"
