File: PCB/AirU/AirU.kicad_sch (KiCad schematic)
At the start: 31 parts, among them IC3 LD1086DT50TR, J1 53261-7008, J2 ZX62-B-5PA_33_, U1 ESP32-S3-WROOM-1, U2 CH340E, U3 LoRa_Breakout, U4 MICS6814, U5 HDC2010YPAR

Commit message: pcb layout complete
Parts:
- added J3, J4, J6: Conn_01x02_Male, Connector_PinHeader_2.54mm:PinHeader_1x02_P2.54mm_Vertical, symbol Connector:Conn_01x02_Male
- added J5: Conn_01x01_Male, Connector_PinHeader_2.54mm:PinHeader_1x01_P2.54mm_Vertical, symbol Connector:Conn_01x01_Male
Connections:
- net GND: now also J4.2 (Pin_2)
- net GPIO18: no longer U4.8 (H)
- net GPIO20: now also J3.2 (Pin_2)
- net GPIO3: now also J3.1 (Pin_1)
- net GPIO8: now also U4.8 (H)
- net U0RXD: now also J6.2 (Pin_2)
- net U0TXD: now also J6.1 (Pin_1)
- net VCC: now also J5.1 (Pin_1)
- net VDD: now also J4.1 (Pin_1)
Other:
- note added: "Test Header Pin Connections"
Changed lines of the file:
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@@
+    (stroke (width 0) (type default) (color 0 0 0 0))
+  )
+  (polyline (pts (xy 207.01 168.91) (xy 289.56 168.91))
     (stroke (width 0) (type default) (color 0 0 0 0))
   )
@@
     (stroke (width 0) (type default) (color 0 0 0 0))
   )
+  (wire (pts (xy 226.06 148.59) (xy 232.41 148.59))
+    (stroke (width 0) (type default) (color 0 0 0 0))
+  )
   (wire (pts (xy 162.56 62.23) (xy 168.91 62.23))
     (stroke (width 0) (type default) (color 0 0 0 0))
@@
     (stroke (width 0) (type default) (color 0 0 0 0))
   )
+  (wire (pts (xy 227.33 137.16) (xy 233.68 137.16))
+    (stroke (width 0) (type default) (color 0 0 0 0))
+  )
   (wire (pts (xy 162.56 46.99) (xy 168.91 46.99))
     (stroke (width 0) (type default) (color 0 0 0 0))
@@
     (stroke (width 0) (type default) (color 0 0 0 0))
   )
+  (wire (pts (xy 227.33 139.7) (xy 233.68 139.7))
+    (stroke (width 0) (type default) (color 0 0 0 0))
+  )
+  (wire (pts (xy 227.33 125.73) (xy 233.68 125.73))
+    (stroke (width 0) (type default) (color 0 0 0 0))
+  )
+  (wire (pts (xy 227.33 158.75) (xy 232.41 158.75))
+    (stroke (width 0) (type default) (color 0 0 0 0))
+  )
   (wire (pts (xy 298.45 74.93) (xy 314.96 74.93))
     (stroke (width 0) (type default) (color 0 0 0 0))
@@
     (stroke (width 0) (type default) (color 0 0 0 0))
   )
+  (polyline (pts (xy 289.56 168.91) (xy 289.56 124.46))
+    (stroke (width 0) (type default) (color 0 0 0 0))
+  )
   (wire (pts (xy 355.6 36.83) (xy 368.3 36.83))
     (stroke (width 0) (type default) (color 0 0 0 0))
@@
     (stroke (width 0) (type default) (color 0 0 0 0))
   )
+  (wire (pts (xy 226.06 151.13) (xy 232.41 151.13))
+    (stroke (width 0) (type default) (color 0 0 0 0))
+  )
   (wire (pts (xy 257.81 26.67) (xy 257.81 29.21))
     (stroke (width 0) (type default) (color 0 0 0 0))
@@
   )
   (wire (pts (xy 384.81 24.13) (xy 389.89 24.13))
+    (stroke (width 0) (type default) (color 0 0 0 0))
+  )
+  (wire (pts (xy 227.33 128.27) (xy 233.68 128.27))
     (stroke (width 0) (type default) (color 0 0 0 0))
   )
@@
     (effects (font (size 3 3)) (justify left bottom))
   )
+  (text "Test Header Pin Connections" (at 212.09 118.11 0)
+    (effects (font (size 1.905 1.905)) (justify left bottom))
+  )
   (text "MICS 6814: NH3, NO2, CO Sensor" (at 15.24 120.65 0)
     (effects (font (size 1.905 1.905)) (justify left bottom))
@@
     (effects (font (size 1.27 1.27)) (justify right bottom))
   )
+  (label "VCC" (at 232.41 158.75 0)
+    (effects (font (size 1.27 1.27)) (justify left bottom))
+  )
   (label "U0TXD" (at 273.05 36.83 0)
     (effects (font (size 1.27 1.27)) (justify left bottom))
@@
     (effects (font (size 1.27 1.27)) (justify left bottom))
   )
+  (label "U0TXD" (at 233.68 125.73 0)
+    (effects (font (size 1.27 1.27)) (justify left bottom))
+  )
   (label "GPIO7" (at 40.64 50.8 180)
     (effects (font (size 1.27 1.27)) (justify right bottom))
@@
     (effects (font (size 1.27 1.27)) (justify right bottom))
   )
+  (label "GPIO20" (at 233.68 139.7 0)
+    (effects (font (size 1.27 1.27)) (justify left bottom))
+  )
   (label "LORA_SCLK" (at 314.96 58.42 90)
     (effects (font (size 1.27 1.27)) (justify left bottom))
@@
     (effects (font (size 1.27 1.27)) (justify right bottom))
   )
+  (label "VDD" (at 232.41 148.59 0)
+    (effects (font (size 1.27 1.27)) (justify left bottom))
+  )
+  (label "GND" (at 232.41 151.13 0)
+    (effects (font (size 1.27 1.27)) (justify left bottom))
+  )
   (label "LORA_SCLK" (at 355.6 31.75 180)
     (effects (font (size 1.27 1.27)) (justify right bottom))
@@
     (effects (font (size 1.27 1.27)) (justify left bottom))
   )
+  (label "GPIO3" (at 233.68 137.16 0)
+    (effects (font (size 1.27 1.27)) (justify left bottom))
+  )
   (label "GPIO2" (at 40.64 38.1 180)
     (effects (font (size 1.27 1.27)) (justify right bottom))
@@
     (effects (font (size 1.27 1.27)) (justify right bottom))
   )
+  (label "U0RXD" (at 233.68 128.27 0)
+    (effects (font (size 1.27 1.27)) (justify left bottom))
+  )
   (label "GPIO47" (at 168.91 54.61 0)
     (effects (font (size 1.27 1.27)) (justify left bottom))
@@
     (effects (font (size 1.27 1.27)) (justify left bottom))
   )
-  (label "GPIO18" (at 39.37 148.59 180)
+  (label "GPIO8" (at 39.37 148.59 180)
     (effects (font (size 1.27 1.27)) (justify right bottom))
   )
@@
     (pin "1")
   )
+  (symbol (lib_id "Connector:Conn_01x02_Male") (at 222.25 137.16 0) (unit 1)
+    (in_bom yes) (on_board yes) (fields_autoplaced)
+    (property "Reference" "J3" (id 0) (at 222.885 132.08 0))
+    (property "Value" "Conn_01x02_Male" (id 1) (at 222.885 134.62 0))
+    (property "Footprint" "Connector_PinHeader_2.54mm:PinHeader_1x02_P2.54mm_Vertical" (id 2) (at 222.25 137.16 0)
+      (effects (font (size 1.27 1.27)) hide)
+    )
+    (property "Datasheet" "~" (id 3) (at 222.25 137.16 0)
+      (effects (font (size 1.27 1.27)) hide)
+    )
+    (pin "1")
+    (pin "2")
+  )
   (symbol (lib_id "53261-7008:53261-7008") (at 379.73 97.79 0) (unit 1)
     (in_bom yes) (on_board yes) (fields_autoplaced)
@@
     (pin "2")
   )
+  (symbol (lib_id "Connector:Conn_01x02_Male") (at 220.98 148.59 0) (unit 1)
+    (in_bom yes) (on_board yes)
+    (property "Reference" "J4" (id 0) (at 221.615 143.51 0))
+    (property "Value" "Conn_01x02_Male" (id 1) (at 222.25 146.05 0))
+    (property "Footprint" "Connector_PinHeader_2.54mm:PinHeader_1x02_P2.54mm_Vertical" (id 2) (at 220.98 148.59 0)
+      (effects (font (size 1.27 1.27)) hide)
+    )
+    (property "Datasheet" "~" (id 3) (at 220.98 148.59 0)
+      (effects (font (size 1.27 1.27)) hide)
+    )
+    (pin "1")
+    (pin "2")
+  )
   (symbol (lib_id "Device:R") (at 59.69 154.94 180) (unit 1)
     (in_bom yes) (on_board yes) (fields_autoplaced)
@@
     (pin "2")
   )
+  (symbol (lib_id "Connector:Conn_01x02_Male") (at 222.25 125.73 0) (unit 1)
+    (in_bom yes) (on_board yes) (fields_autoplaced)
+    (property "Reference" "J6" (id 0) (at 222.885 120.65 0))
+    (property "Value" "Conn_01x02_Male" (id 1) (at 222.885 123.19 0))
+    (property "Footprint" "Connector_PinHeader_2.54mm:PinHeader_1x02_P2.54mm_Vertical" (id 2) (at 222.25 125.73 0)
+      (effects (font (size 1.27 1.27)) hide)
+    )
+    (property "Datasheet" "~" (id 3) (at 222.25 125.73 0)
+      (effects (font (size 1.27 1.27)) hide)
+    )
+    (pin "1")
+    (pin "2")
+  )
   (symbol (lib_id "power:VCC") (at 199.39 90.17 180) (unit 1)
     (in_bom yes) (on_board yes) (fields_autoplaced)
@@
     )
     (property "Datasheet" "" (id 3) (at 372.11 115.57 0)
+      (effects (font (size 1.27 1.27)) hide)
+    )
+    (pin "1")
+  )
+  (symbol (lib_id "Connector:Conn_01x01_Male") (at 222.25 158.75 0) (unit 1)
+    (in_bom yes) (on_board yes) (fields_autoplaced)
+    (property "Reference" "J5" (id 0) (at 222.885 153.67 0))
+    (property "Value" "Conn_01x01_Male" (id 1) (at 222.885 156.21 0))
+    (property "Footprint" "Connector_PinHeader_2.54mm:PinHeader_1x01_P2.54mm_Vertical" (id 2) (at 222.25 158.75 0)
+      (effects (font (size 1.27 1.27)) hide)
+    )
+    (property "Datasheet" "~" (id 3) (at 222.25 158.75 0)
       (effects (font (size 1.27 1.27)) hide)
     )
@@
       (reference "J2") (unit 1) (value "ZX62-B-5PA_33_") (footprint "ZX62-B-5PA_33_:ZX62B5PA33")
     )
+    (path "/71df1879-5202-40c2-bb6a-e8a7a96c5250"
+      (reference "J3") (unit 1) (value "Conn_01x02_Male") (footprint "Connector_PinHeader_2.54mm:PinHeader_1x02_P2.54mm_Vertical")
+    )
+    (path "/a123d48d-57cb-4146-ba3e-4fa29d6f51ab"
+      (reference "J4") (unit 1) (value "Conn_01x02_Male") (footprint "Connector_PinHeader_2.54mm:PinHeader_1x02_P2.54mm_Vertical")
+    )
+    (path "/cacccb5f-65ae-490c-b51e-4855ab288701"
+      (reference "J5") (unit 1) (value "Conn_01x01_Male") (footprint "Connector_PinHeader_2.54mm:PinHeader_1x01_P2.54mm_Vertical")
+    )
+    (path "/b27f272d-42d2-47db-aa2c-5f2e2a1ead69"
+      (reference "J6") (unit 1) (value "Conn_01x02_Male") (footprint "Connector_PinHeader_2.54mm:PinHeader_1x02_P2.54mm_Vertical")
+    )
     (path "/bdd33319-5007-4dae-9bf6-27b9b5e71c09"
